Commit message: change urdf .dae to .stl

File: RobotConfigs/mycobot_pro600/mycobot_pro600.urdf (robot description, URDF)
Before this commit: robot mycobotpro600, 7 links, 6 joints
Links:
- link base: geometry collision mesh filename=meshes/base.stl; visual mesh filename=meshes/base.stl
- link link1: geometry collision mesh filename=meshes/link1.stl; visual mesh filename=meshes/link1.stl
- link link2: geometry collision mesh filename=meshes/link2.stl; visual mesh filename=meshes/link2.stl
- link link3: geometry collision mesh filename=meshes/link3.stl; visual mesh filename=meshes/link3.stl
- link link4: geometry collision mesh filename=meshes/link4.stl; visual mesh filename=meshes/link4.stl
- link link5: geometry collision mesh filename=meshes/link5.stl; visual mesh filename=meshes/link5.stl
- link link6: geometry collision mesh filename=meshes/link6.stl; visual mesh filename=meshes/link6.stl
