Commit message: add: implement main functionality for robot control and digital twin simulation

File: digital_twin/sim/model/static/ElephantRobotics/mycobot_pro600/mycobot_pro600.urdf (robot description, URDF)
Before this commit: robot mycobotpro600, 7 links, 6 joints
Links:
- link base: geometry collision mesh filename=base.stl; visual mesh filename=base.stl
- link link1: geometry collision mesh filename=link1.stl; visual mesh filename=link1.stl
- link link2: geometry collision mesh filename=link2.stl; visual mesh filename=link2.stl
- link link3: geometry collision mesh filename=link3.stl; visual mesh filename=link3.stl
- link link4: geometry collision mesh filename=link4.stl; visual mesh filename=link4.stl
- link link5: geometry collision mesh filename=link5.stl; visual mesh filename=link5.stl
- link link6: geometry collision mesh filename=link6.stl; visual mesh filename=link6.stl

Commit message: fix: update URDF subproject commit and improve robot movement handling in main.py

File: digital_twin/sim/model/static/ElephantRobotics/mycobot_pro600/mycobot_pro600.urdf (robot description, URDF)
Before this commit: robot Elephant Robotics myCobot pro600, 7 links, 6 joints
Joints:
- joint joint2_to_joint1: limit lower=-3.14 upper=3.14159 effort=1000.0 velocity=0 -> lower=-3.14 upper=3.14159 effort=1000.0 velocity=1.0
